File: output/pcbs/reversible.kicad_pcb (KiCad board)
At the start: 2 copper layers, 149.1 x 121.9 mm, 72 parts

Commit message: More overhaul. TODO: Need to renet the pins.
Parts:
- removed REF**: EVQWGD001, RollerEncoder_Panasonic_EVQWGD001
- added ?: EVQWGD001, RollerEncoder_Panasonic_EVQWGD001, F.Cu at (166.5, 73.0)
- moved JST1 57.0 mm to (178.5, 45.5), turned to 0 degrees
- moved DISP1 22.8 mm to (164.5, 39.5)
- moved D30 20.1 mm to (166.5, 65.5), turned to 180 degrees
- moved D29 19.5 mm to (177.5, 120.6), turned to 155 degrees
- moved D28 16.9 mm to (159.8, 112.3), turned to 155 degrees
- moved S29 15.6 mm to (168.4, 125.8), turned to 65 degrees
- moved MH1 14.5 mm to (174.8, 112.2), turned to 65 degrees
- moved D27 13.9 mm to (150.0, 40.0), turned to 90 degrees
- moved D26 13.6 mm to (150.0, 58.5), turned to 90 degrees
- moved D25 13.3 mm to (150.0, 77.0), turned to 90 degrees
- moved D23 13.2 mm to (130.5, 37.0), turned to 90 degrees
- moved D24 13.1 mm to (150.0, 95.5), turned to 90 degrees
- moved D22 12.9 mm to (130.5, 55.5), turned to 90 degrees
- moved S28 12.7 mm to (150.8, 117.5), turned to 65 degrees
- moved D21 12.6 mm to (130.5, 74.0), turned to 90 degrees
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Other:
- board size 149.1 x 121.9 mm -> 159.5 x 127.3 mm

Commit message: Starting to wire the reversible PCB
Parts:
- moved DISP1 0.09 mm to (164.4, 39.5)
- moved MCU1 0.09 mm to (164.4, 35.5)
Connections:
- ? pad A: P006 -> P1
- ? pad C: P008 -> P0
- ? pad S1: P011 -> P7
- D1 pad 1: P115 -> P8
- D10 pad 1: P115 -> P8
- D11 pad 1: P002 -> P9
- D12 pad 1: P029 -> P10
- D13 pad 1: P031 -> P16
- D14 pad 1: P113 -> P7
- D15 pad 1: P115 -> P8
- D16 pad 1: P002 -> P9
- D17 pad 1: P029 -> P10
- D18 pad 1: P031 -> P16
- D19 pad 1: P113 -> P7
- D2 pad 1: P002 -> P9
- D20 pad 1: P115 -> P8
- D21 pad 1: P002 -> P9
- D22 pad 1: P029 -> P10
- D23 pad 1: P031 -> P16
- D24 pad 1: P115 -> P8
- D25 pad 1: P002 -> P9
- D26 pad 1: P029 -> P10
- D27 pad 1: P031 -> P16
- D28 pad 1: P113 -> P7
- D29 pad 1: P113 -> P7
- D3 pad 1: P029 -> P10
- D30 pad 1: P113 -> P21
- D4 pad 1: P031 -> P16
- D5 pad 1: P115 -> P8
- D6 pad 1: P002 -> P9
- D7 pad 1: P029 -> P10
- D8 pad 1: P031 -> P16
- D9 pad 1: P113 -> P7
- DISP1 pad 14: CS -> P2
- DISP1 pad 16: SCK -> P3
- DISP1 pad 17: MOSI -> P4
- DISP1 pad 24: CS -> P2
- DISP1 pad 26: SCK -> P3
- DISP1 pad 27: MOSI -> P4
- S1 pad 2: P011 -> outer_bottom
- S10 pad 2: P106 -> ring_bottom
- S11 pad 2: P106 -> ring_home
- S12 pad 2: P106 -> ring_top
- S13 pad 2: P106 -> ring_num
- S14 pad 2: P106 -> middle_mod
- S15 pad 2: P111 -> middle_bottom
- S16 pad 2: P111 -> middle_home
- S17 pad 2: P111 -> middle_top
- S18 pad 2: P111 -> middle_num
- S19 pad 2: P111 -> index_mod
- S2 pad 2: P011 -> outer_home
- S20 pad 2: P010 -> index_bottom
- S21 pad 2: P010 -> index_home
- S22 pad 2: P010 -> index_top
- S23 pad 2: P010 -> index_num
- S24 pad 2: P009 -> inner_bottom
- S25 pad 2: P009 -> inner_home
- S26 pad 2: P009 -> inner_top
- S27 pad 2: P009 -> inner_num
- S28 pad 2: P010 -> space_cluster
- S29 pad 2: P009 -> extra_cluster
- S3 pad 2: P011 -> outer_top
- S4 pad 2: P011 -> outer_num
- S5 pad 2: P104 -> pinky_bottom
- S6 pad 2: P104 -> pinky_home
- S7 pad 2: P104 -> pinky_top
- S8 pad 2: P104 -> pinky_num
- S9 pad 2: P104 -> ring_mod
Routing:
- net (no net): track 337.7 -> 0.00 mm
- net P14: track 0.00 -> 193.1 mm
- net P16: track 0.00 -> 115.8 mm
- net GND: track 3.50 -> 103.6 mm, vias 0 -> 3
- net P3: track 0.00 -> 78.5 mm, vias 0 -> 2
- net P2: track 0.00 -> 76.5 mm, vias 0 -> 1
- net P4: track 0.00 -> 64.8 mm, vias 0 -> 2
- net RAW: track 0.00 -> 46.2 mm, vias 0 -> 1
- net VCC: track 0.00 -> 38.4 mm
- net outer_num: track 0.00 -> 38.0 mm
- net BAT_P: track 0.00 -> 25.7 mm, vias 0 -> 1
- net P21: track 0.00 -> 9.84 mm
- net P20: track 0.00 -> 9.84 mm
- net P19: track 0.00 -> 9.84 mm
- net P18: track 0.00 -> 9.84 mm
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Other:
- board text added: "Designed by Daniel Fox."
- board text added: "Licensed under the GNU GPLv3."
- board text added: "WayWayWay"
